File: KiCad/io_board/SD drive.sch (KiCad schematic (older format))
At the start: 0 parts

Commit message: Updated IO board schematics and board.
Parts:
- added C17: 100µ, symbol Device:CP
- added C18: 100n, symbol Device:C
- added J3: SD_Card, Connector_Card:SD_Kyocera_145638109211859+, symbol Connector:SD_Card
- added U12: AMS1117-3.3, Package_TO_SOT_SMD:SOT-223-3_TabPin2, symbol Regulator_Linear:AMS1117-3.3
- added U14: 74HC32, symbol 74xx:74LS32
- added U7: EPM240M100, Package_BGA:BGA-100_6.0x6.0mm_Layout11x11_P0.5mm_Ball0.3mm_Pad0.25mm_NSMD, symbol CPLD_Altera:EPM240M100
- added X2: 10 MHz, Oscillator:Oscillator_DIP-14, symbol Oscillator:CXO_DIP14
Connections:
- net labels added: A0, A[0..19], CARD_DET, CPLD_CLK, CS, DI, DO, GND, RA0, RA1, RA2, RA3, RA4, RA5, RA6, RA7, RA8, RA[0..8], RD0, RD1, RD2, RD3, RD4, RD5, RD6, RD7, RD[0..7], SCLK, SD_BUSY, SD_CS, SD_DO, SD_SCLK, VCC, VCC3, ~CS_DRIVE, ~RD, ~RESET, ~WR, ~WR_BUFFER
- wire segments 0 -> 96
- no-connect marks 0 -> 8
