File: KiCad/io_board/io_board.sch (KiCad schematic (older format))
At the start: 0 parts

Commit message: Working on IO board
Changed lines of the file:
@@
 $Descr A4 11693 8268
 encoding utf-8
-Sheet 1 7
+Sheet 1 8
 Title "Mini8086 I/O board"
 Date "2020-11-05"
@@
 F1 "misc.sch" 50
 $EndSheet
+$Sheet
+S 8500 1000 1000 1000
+U 5FAD75B9
+F0 "I2C" 50
+F1 "I2C.sch" 50
+$EndSheet
 $EndSCHEMATC
