File: KiCad/io_board/io_board.kicad_pcb (KiCad board)
At the start: 2 copper layers, 30 parts, among them J1 RS232, J2 Mini-DIN-6, J3 SD_Card, U1 16550, U2 MAX232, U3 SN74LS07N, U4 74HC04, U5 8042, U6 27C512, X1 Edge72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

Commit message: Worked on I/O board.
Parts:
- added C17: 100µ, Capacitor_THT:CP_Radial_D5.0mm_P2.50mm, F.Cu at (231.4, 38.4)
- added C18: 100n, Capacitor_THT:C_Disc_D4.3mm_W1.9mm_P5.00mm, F.Cu at (222.7, 40.3)
- added C19: 100n, Capacitor_THT:C_Disc_D4.3mm_W1.9mm_P5.00mm, F.Cu at (196.3, 50.6)
- added C20: 100n, Capacitor_THT:C_Disc_D4.3mm_W1.9mm_P5.00mm, F.Cu at (196.3, 47.2)
- added C21: 100n, Capacitor_THT:C_Disc_D4.3mm_W1.9mm_P5.00mm, F.Cu at (222.7, 36.8)
- added C22: 100n, Capacitor_THT:C_Disc_D4.3mm_W1.9mm_P5.00mm, F.Cu at (214.6, 40.3)
- added C23: 100n, Capacitor_THT:C_Disc_D4.3mm_W1.9mm_P5.00mm, F.Cu at (214.6, 36.8)
- added C24: 100n, Capacitor_THT:C_Disc_D4.3mm_W1.9mm_P5.00mm, F.Cu at (134.6, 139.1)
- added C25: 100n, Capacitor_THT:C_Disc_D4.3mm_W1.9mm_P5.00mm, F.Cu at (117.9, 106.2)
- added R4: 6K8, Resistor_THT:R_Axial_DIN0207_L6.3mm_D2.5mm_P7.62mm_Horizontal, F.Cu at (172.7, 63.5)
- added R5: 6K8, Resistor_THT:R_Axial_DIN0207_L6.3mm_D2.5mm_P7.62mm_Horizontal, F.Cu at (172.7, 74.2)
- added R6: 4K7, Resistor_THT:R_Axial_DIN0207_L6.3mm_D2.5mm_P7.62mm_Horizontal, F.Cu at (160.5, 147.3)
- added U10: 74HC367, Package_SO:SOIC-16_4.55x10.3mm_P1.27mm, F.Cu at (99.1, 102.6)
- added U11: 74HC367, Package_SO:SOIC-16_4.55x10.3mm_P1.27mm, F.Cu at (98.6, 88.4)
- added U12: AMS1117-3.3, Package_TO_SOT_SMD:SOT-223-3_TabPin2, F.Cu at (125.0, 103.6)
- added U13: SN74LVC245A, Package_SO:TSSOP-20_4.4x6.5mm_P0.65mm, F.Cu at (124.5, 130.0)
- added U14: 74HCT32, Package_SO:SOIC-14_3.9x8.7mm_P1.27mm, F.Cu at (124.5, 116.8)
- added U15: SN74LVC8T245PWR, Package_SO:TSSOP-24_4.4x7.8mm_P0.65mm, F.Cu at (124.5, 142.2)
- added U4: 74HC04, Package_SO:SOIC-14_3.9x8.7mm_P1.27mm, F.Cu at (75.2, 88.4)
- added U7: EPM240T100, Package_QFP:LQFP-100_14x14mm_P0.5mm, F.Cu at (146.8, 136.1)
- added U8: 74HC245, Package_SO:SOIC-20W_7.5x12.8mm_P1.27mm, F.Cu at (146.3, 115.8)
- added U9: 62256, Package_DIP:DIP-28_W7.62mm_LongPads, F.Cu at (95.5, 113.8)
- added X2: 10 MHz, Oscillator:Oscillator_DIP-14, F.Cu at (138.7, 104.1)
- C16: footprint Capacitor_THT:CP_Radial_D6.3mm_P2.50mm -> Capacitor_THT:CP_Radial_D5.0mm_P2.00mm
- U1: footprint Package_DIP:DIP-40_W15.24mm -> Package_DIP:DIP-40_W15.24mm_Socket_LongPads
- U3: value SN74LS07N -> 74HC07
- U6: footprint Package_DIP:DIP-28_W15.24mm -> Package_DIP:DIP-28_W15.24mm_Socket_LongPads
- moved U6 190.6 mm to (49.8, 58.4)
- moved U4 149.5 mm to (72.6, 58.4)
- moved U3 146.3 mm to (87.9, 58.4)
- moved C8 96.8 mm to (177.8, 55.9), turned to 270 degrees
- moved C9 87.6 mm to (177.8, 63.5), turned to 90 degrees
- moved J2 85.3 mm to (185.9, 63.0), turned to 90 degrees
- moved U1 81.7 mm to (72.6, 98.6)
- moved C7 80.8 mm to (177.8, 68.6), turned to 90 degrees
- moved U5 68.8 mm to (49.8, 98.6), turned to 0 degrees
- moved C2 44.0 mm to (120.3, 86.5)
- moved C5 44.0 mm to (120.8, 81.6)
- moved C6 44.0 mm to (127.5, 81.6)
- moved R1 44.0 mm to (120.3, 76.3)
- moved R2 44.0 mm to (120.3, 72.2)
- moved Y1 44.0 mm to (122.7, 66.9)
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Connections:
- net Net-(X1-Pad16) renamed A11
- net Net-(X1-Pad17) renamed A12
- net Net-(X1-Pad18) renamed A13
- net Net-(X1-Pad19) renamed A14
- net Net-(X1-Pad20) renamed A15
- net Net-(X1-Pad21) renamed A16
- net Net-(X1-Pad22) renamed A17
- net Net-(X1-Pad23) renamed A18
- net Net-(X1-Pad24) renamed A19
- J3 pad 1: Net-(J3-Pad1) -> /SD drive/SD_CS
- J3 pad 10: Net-(J3-Pad10) -> CARD_DET
- J3 pad 12: Net-(J3-Pad12) -> GND
- J3 pad 13: Net-(J3-Pad13) -> GND
- J3 pad 2: Net-(J3-Pad2) -> /SD drive/SD_DI
- J3 pad 3: Net-(J3-Pad3) -> GND
- J3 pad 4: Net-(J3-Pad4) -> VCC3
- J3 pad 5: Net-(J3-Pad5) -> /SD drive/SD_SCLK
- J3 pad 6: Net-(J3-Pad6) -> GND
- J3 pad 7: Net-(J3-Pad7) -> /SD drive/SD_DO
- U1 pad 1: Net-(U1-Pad1) -> D0
- U1 pad 2: Net-(U1-Pad2) -> D1
- U1 pad 3: Net-(U1-Pad3) -> D2
- U1 pad 4: Net-(U1-Pad4) -> D3
- U1 pad 5: Net-(U1-Pad5) -> D4
- U1 pad 6: Net-(U1-Pad6) -> D5
- U1 pad 7: Net-(U1-Pad7) -> D6
- U1 pad 8: Net-(U1-Pad8) -> D7
- U6 pad 15: Net-(U6-Pad15) -> ~CS_BUFFER
- U6 pad 26: GND -> ~WR
- U6 pad 27: GND -> ~RD
- X1 pad 10: Net-(X1-Pad10) -> A5
- X1 pad 11: Net-(X1-Pad11) -> A6
- X1 pad 12: Net-(X1-Pad12) -> A7
- X1 pad 13: Net-(X1-Pad13) -> A8
- X1 pad 14: Net-(X1-Pad14) -> A9
- X1 pad 15: Net-(X1-Pad15) -> A10
- X1 pad 5: Net-(X1-Pad5) -> A0
- X1 pad 6: Net-(X1-Pad6) -> A1
- X1 pad 7: Net-(X1-Pad7) -> A2
- X1 pad 8: Net-(X1-Pad8) -> A3
- X1 pad 9: Net-(X1-Pad9) -> A4
Routing:
- added copper zone on In2.Cu, net GND
Other:
- board outline added: 160.3 x 99.1 mm
- copper layers 2 -> 4
- net class Default: trace_width 0.25 -> 0.2; via_dia 0.8 -> 0.45; via_drill 0.4 -> 0.2
- rule via_min_drill: 0.3 -> 0.2
- rule via_min_size: 0.4 -> 0.45

Commit message: Working on IO board
Parts:
- added C26: 100n, Capacitor_SMD:C_1206_3216Metric, F.Cu at (156.3, 70.5)
- added C27: 100n, Capacitor_SMD:C_1206_3216Metric, F.Cu at (156.3, 73.8)
- added J4: JTAG, Connector_IDC:IDC-Header_2x05_P2.54mm_Vertical, F.Cu at (118.7, 62.2)
- added R7: 1K, Resistor_THT:R_Axial_DIN0207_L6.3mm_D2.5mm_P7.62mm_Horizontal, F.Cu at (144.3, 64.8)
- added R8: 10K, Resistor_THT:R_Axial_DIN0207_L6.3mm_D2.5mm_P7.62mm_Horizontal, F.Cu at (140.8, 64.8)
- added R9: 10K, Resistor_THT:R_Axial_DIN0207_L6.3mm_D2.5mm_P7.62mm_Horizontal, F.Cu at (137.4, 64.8)
- added U16: MAX485E, Package_DIP:DIP-8_W7.62mm_LongPads, F.Cu at (129.5, 70.9)
- C1, C2: value 22p -> 27p
- C10, C11, C25: footprint Capacitor_THT:C_Disc_D4.3mm_W1.9mm_P5.00mm -> Capacitor_SMD:C_1206_3216Metric
- C18: footprint Capacitor_THT:C_Disc_D4.3mm_W1.9mm_P5.00mm -> Capacitor_THT:C_Disc_D3.0mm_W2.0mm_P2.50mm
- C21, C22, C23, C24: footprint Capacitor_THT:C_Disc_D4.3mm_W1.9mm_P5.00mm -> Capacitor_SMD:C_1206_3216Metric; moved to B.Cu
- R1: value 10M -> 1M
- R2: value 470 -> 47
- U1: value 16550 -> ST16C550CJ44; footprint Package_DIP:DIP-40_W15.24mm_Socket_LongPads -> Package_LCC:PLCC-44_THT-Socket
- U4: value 74HC04 -> 74HCT04
- moved C16 235.3 mm to (45.2, 142.7), turned to 270 degrees
- moved C14 198.0 mm to (69.0, 58.5), turned to 270 degrees
- moved C15 172.2 mm to (91.3, 98.7), turned to 270 degrees
- moved C12 158.6 mm to (101.3, 81.0), turned to 180 degrees
- moved C11 155.8 mm to (111.3, 57.9), turned to 270 degrees
- moved C20 144.3 mm to (60.2, 95.1), turned to 180 degrees
- moved C18 132.1 mm to (120.8, 124.3)
- moved C1 127.3 mm to (83.3, 88.6)
- moved C21 122.7 mm to (150.6, 136.1), turned to 270 degrees
- moved C22 121.2 mm to (146.8, 140.7), turned to 180 degrees
- moved C17 118.1 mm to (133.0, 103.6)
- moved C23 116.3 mm to (146.8, 131.3)
- moved C10 115.4 mm to (154.9, 115.8), turned to 90 degrees
- moved C19 109.6 mm to (106.7, 113.8), turned to 270 degrees
- moved C13 101.0 mm to (177.7, 85.3), turned to 270 degrees
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Connections:
- U1 pad 1: D0 -> (no net)
- U1 pad 12: VCC -> (no net)
- U1 pad 13: VCC -> Net-(U1-Pad13)
- U1 pad 14: ~CS_UART -> VCC
- U1 pad 15: Net-(U1-Pad15) -> VCC
- U1 pad 16: Net-(C1-Pad1) -> ~CS_UART
- U1 pad 17: Net-(R2-Pad2) -> Net-(U1-Pad10)
- U1 pad 18: ~WR -> Net-(C1-Pad1)
- U1 pad 19: GND -> Net-(R2-Pad2)
- U1 pad 2: D1 -> D0
- U1 pad 20: GND -> ~WR
- U1 pad 21: ~RD -> GND
- U1 pad 23: Net-(U1-Pad23) -> (no net)
- U1 pad 24: Net-(U1-Pad24) -> GND
- U1 pad 25: GND -> ~RD
- U1 pad 26: A2 -> Net-(U1-Pad26)
- U1 pad 27: A1 -> Net-(U1-Pad27)
- U1 pad 28: A0 -> GND
- U1 pad 29: Net-(U1-Pad29) -> A2
- U1 pad 3: D2 -> D1
- U1 pad 30: IRQ4 -> A1
- U1 pad 31: Net-(U1-Pad31) -> A0
- U1 pad 33: Net-(U1-Pad33) -> IRQ4
- U1 pad 34: Net-(U1-Pad34) -> (no net)
- U1 pad 35: RESET -> Net-(U1-Pad35)
- U1 pad 37: VCC -> Net-(U1-Pad37)
- U1 pad 38: VCC -> Net-(U1-Pad38)
- U1 pad 39: VCC -> RESET
- U1 pad 4: D3 -> D2
- U1 pad 40: VCC -> Net-(U1-Pad40)
- U1 pad 5: D4 -> D3
- U1 pad 6: D5 -> D4
- U1 pad 7: D6 -> D5
- U1 pad 8: D7 -> D6
- U1 pad 9: Net-(U1-Pad15) -> D7
- U2 pad 10: Net-(U1-Pad32) -> Net-(U1-Pad36)
- U2 pad 11: Net-(U1-Pad11) -> Net-(U1-Pad13)
- U2 pad 12: Net-(U1-Pad10) -> Net-(U1-Pad11)
- U2 pad 9: Net-(U1-Pad36) -> Net-(U1-Pad40)
- U3 pad 14: (no net) -> VCC
- U3 pad 7: (no net) -> GND
- U4 pad 10: Net-(U4-Pad10) -> /connector/IRQ7
- U4 pad 11: GND -> ~INT_I2C
- U7 pad 22: Net-(U7-Pad22) -> /SD drive/TMS
- U7 pad 23: Net-(U7-Pad23) -> /SD drive/TDI
- U7 pad 24: Net-(U7-Pad24) -> /SD drive/TCK
- U7 pad 25: Net-(U7-Pad25) -> /SD drive/TDO
- X1 pad 62: Net-(X1-Pad62) -> /connector/IRQ7
Routing:
- net GND: track 0.00 -> 65.0 mm, vias 0 -> 12
- net VCC: track 0.00 -> 37.6 mm, vias 0 -> 4
- added copper zone on F.Cu, net GND

Commit message: Worked on I/O board.
Parts:
- removed the U4 at (104.0, 61.5)
- removed the U4 at (72.6, 58.4)
- added C28: 10n, Capacitor_THT:C_Disc_D4.3mm_W1.9mm_P5.00mm, F.Cu at (161.5, 143.5)
- added C29: 100n, Capacitor_SMD:C_1206_3216Metric, B.Cu at (113.5, 86.1)
- added J5: DS1307, Connector_PinHeader_2.54mm:PinHeader_1x04_P2.54mm_Vertical, F.Cu at (143.5, 19.8)
- added J6: BME280, Connector_PinHeader_2.54mm:PinHeader_1x04_P2.54mm_Vertical, F.Cu at (148.2, 19.8)
- added R10: 1K8, Resistor_THT:R_Axial_DIN0207_L6.3mm_D2.5mm_P2.54mm_Vertical, F.Cu at (121.7, 84.8)
- added R11: 1K8, Resistor_THT:R_Axial_DIN0207_L6.3mm_D2.5mm_P2.54mm_Vertical, F.Cu at (121.7, 92.5)
- added U17: PCA9564D, Package_SO:SOIC-20W_7.5x12.8mm_P1.27mm, F.Cu at (113.5, 90.2)
- added U18: 24C04, Package_SO:SOIC-8_3.9x4.9mm_P1.27mm, F.Cu at (117.1, 75.9)
- added U19: SN74AVC8T245PW, Package_SO:TSSOP-24_4.4x7.8mm_P0.65mm, F.Cu at (100.6, 91.7)
- added U4: 74HCT04, Package_SO:SOIC-14_3.9x8.7mm_P1.27mm, F.Cu at (75.2, 125.1)
- C10, C11, C26, C27: moved to B.Cu
- R1, R2, R3, R4, R5, R6, R8, R9: footprint Resistor_THT:R_Axial_DIN0207_L6.3mm_D2.5mm_P7.62mm_Horizontal -> Resistor_THT:R_Axial_DIN0207_L6.3mm_D2.5mm_P2.54mm_Vertical
- R7: value 1K -> 2K2; footprint Resistor_THT:R_Axial_DIN0207_L6.3mm_D2.5mm_P7.62mm_Horizontal -> Resistor_THT:R_Axial_DIN0207_L6.3mm_D2.5mm_P2.54mm_Vertical
- moved U16 104.6 mm to (215.4, 11.2)
- moved J4 86.5 mm to (138.9, 146.3)
- moved C27 77.6 mm to (104.1, 131.2), turned to 90 degrees
- moved C11 76.1 mm to (75.2, 125.0)
- moved C12 76.1 mm to (174.8, 61.0), turned to 270 degrees
- moved R9 74.9 mm to (149.6, 138.7), turned to 180 degrees
- moved R7 74.1 mm to (138.9, 138.7), turned to 180 degrees
- moved R8 74.0 mm to (144.3, 138.7), turned to 180 degrees
- moved C17 73.4 mm to (73.4, 146.6)
- moved R3 69.4 mm to (108.7, 58.4)
- moved C5 67.2 mm to (98.6, 80.6)
- moved C13 67.2 mm to (114.7, 62.0)
- moved C3 67.2 mm to (98.6, 60.6)
- moved C4 67.2 mm to (98.6, 72.3)
- moved C6 67.2 mm to (98.6, 69.0)
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Connections:
- net Net-(U15-Pad14) renamed /SD drive/D7_3
- net Net-(U15-Pad15) renamed /SD drive/D6_3
- net Net-(U15-Pad16) renamed /SD drive/D5_3
- net Net-(U15-Pad17) renamed /SD drive/D4_3
- net Net-(U15-Pad18) renamed /SD drive/D3_3
- net Net-(U15-Pad19) renamed /SD drive/D2_3
- net Net-(U15-Pad20) renamed /SD drive/D1_3
- net Net-(U15-Pad21) renamed /SD drive/D0_3
- R8 pad 2: GND -> VCC
- R9 pad 2: GND -> VCC
- U1 pad 1: (no net) -> Net-(U1-Pad1)
- U1 pad 12: (no net) -> Net-(U1-Pad12)
- U1 pad 23: (no net) -> Net-(U1-Pad23)
- U1 pad 34: (no net) -> Net-(U1-Pad34)
- U6 pad 16: Net-(U6-Pad16) -> ~CS_I2C
Routing:
- added copper zone on B.Cu, net GND

Commit message: Continued work on I/O board.
Parts:
- added C30: 100n, Capacitor_SMD:C_1206_3216Metric, B.Cu at (111.3, 102.6)
- added C31: 100n, Capacitor_SMD:C_1206_3216Metric, B.Cu at (100.6, 102.6)
- added C32: 100n, Capacitor_SMD:C_1206_3216Metric, B.Cu at (97.8, 91.4)
- added C33: 100n, Capacitor_SMD:C_1206_3216Metric, B.Cu at (57.4, 137.2)
- added C34: 100n, Capacitor_SMD:C_1206_3216Metric, B.Cu at (79.8, 67.1)
- added C35: 100n, Capacitor_SMD:C_1206_3216Metric, B.Cu at (89.0, 102.7)
- added C36: 100n, Capacitor_SMD:C_1206_3216Metric, B.Cu at (88.6, 119.3)
- added C37: 100n, Capacitor_SMD:C_1206_3216Metric, B.Cu at (115.6, 78.1)
- added C38: 100n, Capacitor_SMD:C_1206_3216Metric, B.Cu at (101.1, 144.5)
- added C39: 100n, Capacitor_SMD:C_1206_3216Metric, B.Cu at (142.9, 132.0)
- C1, C2: footprint Capacitor_THT:C_Disc_D3.0mm_W1.6mm_P2.50mm -> Capacitor_SMD:C_1206_3216Metric; moved to B.Cu
- C12, C19, C28: footprint Capacitor_THT:C_Disc_D4.3mm_W1.9mm_P5.00mm -> Capacitor_SMD:C_1206_3216Metric
- C13, C14, C15, C20: footprint Capacitor_THT:C_Disc_D4.3mm_W1.9mm_P5.00mm -> Capacitor_SMD:C_1206_3216Metric; moved to B.Cu
- C18: footprint Capacitor_THT:C_Disc_D3.0mm_W2.0mm_P2.50mm -> Capacitor_SMD:C_1206_3216Metric
- C7, C8, C9: footprint Capacitor_THT:C_Disc_D3.0mm_W1.6mm_P2.50mm -> Capacitor_SMD:C_1206_3216Metric
- R1, R10, R11, R2: footprint Resistor_THT:R_Axial_DIN0207_L6.3mm_D2.5mm_P2.54mm_Vertical -> Resistor_SMD:R_1206_3216Metric; moved to B.Cu
- R3, R4, R5, R6, R7, R8, R9: footprint Resistor_THT:R_Axial_DIN0207_L6.3mm_D2.5mm_P2.54mm_Vertical -> Resistor_SMD:R_1206_3216Metric
- U2: footprint Package_DIP:DIP-16_W7.62mm_LongPads -> Package_SO:SOIC-16_3.9x9.9mm_P1.27mm
- moved C10 16.1 mm to (126.5, 139.2), turned to 270 degrees
- moved C13 9.94 mm to (106.6, 67.7)
- moved U2 9.12 mm to (106.6, 70.6)
- moved R3 5.87 mm to (104.1, 62.1), turned to 270 degrees
- moved C15 5.23 mm to (75.4, 101.6), turned to 270 degrees
- moved R11 4.70 mm to (118.0, 89.5)
- moved C14 4.66 mm to (58.7, 60.8)
- moved C20 4.09 mm to (59.2, 100.3)
- moved R10 3.70 mm to (118.0, 84.5)
- moved C19 3.05 mm to (75.4, 132.2)
- moved R1 2.82 mm to (83.1, 90.0)
- moved C24 2.80 mm to (103.6, 117.7)
- moved U18 2.64 mm to (115.6, 78.1), turned to 0 degrees
- moved R2 2.54 mm to (72.8, 86.9), turned to 270 degrees
- moved C12 2.54 mm to (174.8, 63.5)
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Connections:
- net Net-(C1-Pad1) renamed /serial/XTAL1
- net Net-(R2-Pad2) renamed /serial/XTAL2
- J4 pad 4: VCC -> VCC3
- R8 pad 2: VCC -> VCC3
- R9 pad 2: VCC -> VCC3
- U14 pad 1: Net-(U14-Pad1) -> GND
- U14 pad 10: Net-(U14-Pad10) -> GND
- U14 pad 12: Net-(U14-Pad12) -> GND
- U14 pad 13: Net-(U14-Pad13) -> GND
- U14 pad 2: Net-(U14-Pad2) -> GND
- U14 pad 9: Net-(U14-Pad9) -> GND
Routing:
- net VCC: track 37.6 -> 561.9 mm, vias 4 -> 12
- net VCC3: track 0.00 -> 251.6 mm, vias 0 -> 16
- net D7: track 0.00 -> 244.5 mm, vias 0 -> 6
- net D0: track 0.00 -> 239.7 mm, vias 0 -> 6
- net ~RD: track 0.00 -> 235.9 mm, vias 0 -> 9
- net D2: track 0.00 -> 234.8 mm, vias 0 -> 6
- net D4: track 0.00 -> 227.3 mm, vias 0 -> 4
- net D1: track 0.00 -> 222.1 mm, vias 0 -> 6
- net D5: track 0.00 -> 221.7 mm, vias 0 -> 4
- net D6: track 0.00 -> 216.5 mm, vias 0 -> 4
- net D3: track 0.00 -> 209.8 mm, vias 0 -> 8
- net A0: track 0.00 -> 202.0 mm, vias 0 -> 6
- net ~WR: track 0.00 -> 195.3 mm, vias 0 -> 7
- net A1: track 0.00 -> 179.7 mm, vias 0 -> 6
- net ~RESET: track 0.00 -> 135.6 mm, vias 0 -> 4
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- added copper zone on In1.Cu, net GND
