File: KiCad/io_board/PS2.sch (KiCad schematic (older format))
At the start: 9 parts, among them J2 Keyboard, U3 74HC07, U4 74HCT04, U5 8042

Commit message: Updated I/O board
Connections:
- net GND: now also J2.2; no longer J2.3
- net KBD_CLK: now also J2.1; no longer J2.5
- net KBD_DATA: now also J2.3; no longer J2.1
- net VCC: now also J2.5; no longer J2.4
- net ~PCLK: now reaches U4.4, U5.3 (X2)
- net KCLK_OUT: now reaches U4.1, U5.37 (P2.6)
- net KDATA_OUT: now reaches U3.3, U5.38 (P2.7)
- net A0 renamed A2
Other:
- note added: "Attention: Mini-DIN 6 footprint pin numbers are wrong.\n"
- moved on the sheet: C7, C8, C9, J2, R4, R5, U3A, U3B, U3G, U4A, U4B, U5
