File: KiCad/io_board/SD misc.sch (KiCad schematic (older format))
At the start: 5 parts, among them U10 74HC367, U11 74HC367, U14 74HC32, U8 74HC245, U9 62256

Commit message: Worked on I/O board.
Parts:
- U10, U11: footprint (none) -> Package_SO:SOIC-16_4.55x10.3mm_P1.27mm
- U14: value 74HC32 -> 74HCT32; footprint (none) -> Package_SO:SOIC-14_3.9x8.7mm_P1.27mm
- U8: footprint (none) -> Package_SO:SOIC-20W_7.5x12.8mm_P1.27mm
- U9: footprint Package_DIP:DIP-28_W15.24mm -> Package_DIP:DIP-28_W7.62mm_LongPads
Connections:
- net SD_BUSY: no longer U14.2
- net ~ACC_BUFFER: now also U8.19 (CE)
- net at U14.3: no longer U8.19 (CE)
- net ~CS_DRVBUF: no longer names the net of U14.1
Other:
- moved on the sheet: U14A, U14C, U14D, U9

Commit message: Working on IO board
Changed lines of the file:
@@
 $Descr A4 11693 8268
 encoding utf-8
-Sheet 5 7
+Sheet 5 8
 Title "Mini8086 I/O board"
 Date "2020-11-05"
@@
 Text Label 3400 2000 0    50   ~ 0
 RD7
-Text GLabel 3700 1150 2    50   Input ~ 0
+Text GLabel 3700 1150 2    50   BiDi ~ 0
 RD[0..7]
-Text GLabel 2000 1150 0    50   Input ~ 0
+Text GLabel 2000 1150 0    50   BiDi ~ 0
 D[0..7]
 Wire Wire Line
@@
 	10300 950  10400 950
 Connection ~ 10300 950
-Text GLabel 10400 950  2    50   Input ~ 0
+Text GLabel 10400 950  2    50   Output ~ 0
 RA[0..8]
 Text Label 8150 1650 0    50   ~ 0

Commit message: Worked on I/O board.
Connections:
- no-connect marks 3 -> 6
Other:
- moved on the sheet: U14A, U14C, U14D
Changed lines of the file:
@@
 L 74xx:74LS32 U?
 U 1 1 5F9F4271
-P 8450 4950
+P 7500 4850
 AR Path="/5F806563/5F9F4271" Ref="U?"  Part="1"
 AR Path="/5F806563/5F9E8365/5F9F4271" Ref="U14"  Part="1"
-F 0 "U14" H 8450 5275 50  0000 C CNN
-F 1 "74HCT32" H 8450 5184 50  0000 C CNN
-F 2 "Package_SO:SOIC-14_3.9x8.7mm_P1.27mm" H 8450 4950 50  0001 C CNN
-F 3 "http://www.ti.com/lit/gpn/sn74LS32" H 8450 4950 50  0001 C CNN
-	1    8450 4950
+F 0 "U14" H 7500 5175 50  0000 C CNN
+F 1 "74HCT32" H 7500 5084 50  0000 C CNN
+F 2 "Package_SO:SOIC-14_3.9x8.7mm_P1.27mm" H 7500 4850 50  0001 C CNN
+F 3 "http://www.ti.com/lit/gpn/sn74LS32" H 7500 4850 50  0001 C CNN
+	1    7500 4850
 	-1   0    0    1
 $EndComp
@@
 L 74xx:74LS32 U?
 U 4 1 5FA6D7A1
-P 9350 4300
+P 8400 4200
 AR Path="/5F806563/5FA6D7A1" Ref="U?"  Part="4"
 AR Path="/5F806563/5F9E8365/5FA6D7A1" Ref="U14"  Part="4"
-F 0 "U14" H 9350 4625 50  0000 C CNN
-F 1 "74HCT32" H 9350 4534 50  0000 C CNN
-F 2 "Package_SO:SOIC-14_3.9x8.7mm_P1.27mm" H 9350 4300 50  0001 C CNN
-F 3 "http://www.ti.com/lit/gpn/sn74LS32" H 9350 4300 50  0001 C CNN
-	4    9350 4300
+F 0 "U14" H 8400 4525 50  0000 C CNN
+F 1 "74HCT32" H 8400 4434 50  0000 C CNN
+F 2 "Package_SO:SOIC-14_3.9x8.7mm_P1.27mm" H 8400 4200 50  0001 C CNN
+F 3 "http://www.ti.com/lit/gpn/sn74LS32" H 8400 4200 50  0001 C CNN
+	4    8400 4200
 	-1   0    0    1
 $EndComp
@@
 L 74xx:74LS32 U14
 U 3 1 5FA8979A
-P 8450 4300
-F 0 "U14" H 8450 4625 50  0000 C CNN
-F 1 "74HCT32" H 8450 4534 50  0000 C CNN
-F 2 "Package_SO:SOIC-14_3.9x8.7mm_P1.27mm" H 8450 4300 50  0001 C CNN
-F 3 "http://www.ti.com/lit/gpn/sn74LS32" H 8450 4300 50  0001 C CNN
-	3    8450 4300
+P 7500 4200
+F 0 "U14" H 7500 4525 50  0000 C CNN
+F 1 "74HCT32" H 7500 4434 50  0000 C CNN
+F 2 "Package_SO:SOIC-14_3.9x8.7mm_P1.27mm" H 7500 4200 50  0001 C CNN
+F 3 "http://www.ti.com/lit/gpn/sn74LS32" H 7500 4200 50  0001 C CNN
+	3    7500 4200
 	-1   0    0    1
 $EndComp
@@
 	3600 2350 6650 2350
 Connection ~ 6650 2350
+NoConn ~ 8100 4200
+NoConn ~ 7200 4200
+NoConn ~ 7200 4850
 Wire Bus Line
 	8700 1100 8700 1750

Commit message: Continued work on I/O board.
Connections:
- net GND: now also U14.1, U14.10, U14.12, U14.13, U14.2, U14.9
Other:
- moved on the sheet: U14A, U14C, U14D
Changed lines of the file:
@@
 L 74xx:74LS32 U?
 U 1 1 5F9F4271
-P 7500 4850
+P 5750 4800
 AR Path="/5F806563/5F9F4271" Ref="U?"  Part="1"
 AR Path="/5F806563/5F9E8365/5F9F4271" Ref="U14"  Part="1"
-F 0 "U14" H 7500 5175 50  0000 C CNN
-F 1 "74HCT32" H 7500 5084 50  0000 C CNN
-F 2 "Package_SO:SOIC-14_3.9x8.7mm_P1.27mm" H 7500 4850 50  0001 C CNN
-F 3 "http://www.ti.com/lit/gpn/sn74LS32" H 7500 4850 50  0001 C CNN
-	1    7500 4850
+F 0 "U14" H 5750 5125 50  0000 C CNN
+F 1 "74HCT32" H 5750 5034 50  0000 C CNN
+F 2 "Package_SO:SOIC-14_3.9x8.7mm_P1.27mm" H 5750 4800 50  0001 C CNN
+F 3 "http://www.ti.com/lit/gpn/sn74LS32" H 5750 4800 50  0001 C CNN
+	1    5750 4800
 	-1   0    0    1
 $EndComp
@@
 L 74xx:74LS32 U?
 U 4 1 5FA6D7A1
-P 8400 4200
+P 5800 3500
 AR Path="/5F806563/5FA6D7A1" Ref="U?"  Part="4"
 AR Path="/5F806563/5F9E8365/5FA6D7A1" Ref="U14"  Part="4"
-F 0 "U14" H 8400 4525 50  0000 C CNN
-F 1 "74HCT32" H 8400 4434 50  0000 C CNN
-F 2 "Package_SO:SOIC-14_3.9x8.7mm_P1.27mm" H 8400 4200 50  0001 C CNN
-F 3 "http://www.ti.com/lit/gpn/sn74LS32" H 8400 4200 50  0001 C CNN
-	4    8400 4200
+F 0 "U14" H 5800 3825 50  0000 C CNN
+F 1 "74HCT32" H 5800 3734 50  0000 C CNN
+F 2 "Package_SO:SOIC-14_3.9x8.7mm_P1.27mm" H 5800 3500 50  0001 C CNN
+F 3 "http://www.ti.com/lit/gpn/sn74LS32" H 5800 3500 50  0001 C CNN
+	4    5800 3500
 	-1   0    0    1
 $EndComp
@@
 L 74xx:74LS32 U14
 U 3 1 5FA8979A
-P 7500 4200
-F 0 "U14" H 7500 4525 50  0000 C CNN
-F 1 "74HCT32" H 7500 4434 50  0000 C CNN
-F 2 "Package_SO:SOIC-14_3.9x8.7mm_P1.27mm" H 7500 4200 50  0001 C CNN
-F 3 "http://www.ti.com/lit/gpn/sn74LS32" H 7500 4200 50  0001 C CNN
-	3    7500 4200
+P 5750 4150
+F 0 "U14" H 5750 4475 50  0000 C CNN
+F 1 "74HCT32" H 5750 4384 50  0000 C CNN
+F 2 "Package_SO:SOIC-14_3.9x8.7mm_P1.27mm" H 5750 4150 50  0001 C CNN
+F 3 "http://www.ti.com/lit/gpn/sn74LS32" H 5750 4150 50  0001 C CNN
+	3    5750 4150
 	-1   0    0    1
 $EndComp
@@
 	3600 2350 6650 2350
 Connection ~ 6650 2350
-NoConn ~ 8100 4200
-NoConn ~ 7200 4200
-NoConn ~ 7200 4850
+NoConn ~ 5500 3500
+NoConn ~ 5450 4150
+NoConn ~ 5450 4800
+Wire Wire Line
+	6050 4050 6150 4050
+Wire Wire Line
+	6150 4050 6150 4250
+Wire Wire Line
+	6150 4900 6050 4900
+Connection ~ 6150 4900
+Wire Wire Line
+	6150 4900 6150 5050
+Wire Wire Line
+	6050 4700 6150 4700
+Connection ~ 6150 4700
+Wire Wire Line
+	6150 4700 6150 4900
+Wire Wire Line
+	6050 4250 6150 4250
+Connection ~ 6150 4250
+Wire Wire Line
+	6150 4250 6150 4700
+Wire Wire Line
+	6100 3600 6150 3600
+Wire Wire Line
+	6150 3600 6150 4050
+Connection ~ 6150 4050
+Wire Wire Line
+	6100 3400 6150 3400
+Wire Wire Line
+	6150 3400 6150 3600
+Connection ~ 6150 3600
+$Comp
+L power:GND #PWR0104
+U 1 1 5FD540A4
+P 6150 5050
+F 0 "#PWR0104" H 6150 4800 50  0001 C CNN
+F 1 "GND" H 6155 4877 50  0000 C CNN
+F 2 "" H 6150 5050 50  0001 C CNN
+F 3 "" H 6150 5050 50  0001 C CNN
+	1    6150 5050
+	1    0    0    -1
+$EndComp
 Wire Bus Line
 	8700 1100 8700 1750

Commit message: Worked on I/O board.
Connections:
- net GND: no longer U14.12, U14.13
- net IRQ6: now reaches U14.11
- net ~CS_BUFFER renamed ~WR_BUFFER
- new net SD_IRQ: U14.12, U14.13
- no-connect marks 6 -> 5
Other:
- moved on the sheet: U14D
Changed lines of the file:
@@
 Wire Wire Line
 	6650 1750 6650 2350
-$Comp
-L 74xx:74LS32 U?
-U 4 1 5FA6D7A1
-P 5800 3500
-AR Path="/5F806563/5FA6D7A1" Ref="U?"  Part="4"
-AR Path="/5F806563/5F9E8365/5FA6D7A1" Ref="U14"  Part="4"
-F 0 "U14" H 5800 3825 50  0000 C CNN
-F 1 "74HCT32" H 5800 3734 50  0000 C CNN
-F 2 "Package_SO:SOIC-14_3.9x8.7mm_P1.27mm" H 5800 3500 50  0001 C CNN
-F 3 "http://www.ti.com/lit/gpn/sn74LS32" H 5800 3500 50  0001 C CNN
-	4    5800 3500
-	-1   0    0    1
-$EndComp
 Text Label 6000 1750 0    50   ~ 0
 ~ACC_BUFFER
 Text GLabel 5300 1850 0    50   Input ~ 0
-~CS_BUFFER
+~WR_BUFFER
 $Comp
 L 74xx:74LS32 U?
@@
 	3600 2350 6650 2350
 Connection ~ 6650 2350
-NoConn ~ 5500 3500
 NoConn ~ 5450 4150
 NoConn ~ 5450 4800
@@
 Wire Wire Line
 	6150 4250 6150 4700
-Wire Wire Line
-	6100 3600 6150 3600
-Wire Wire Line
-	6150 3600 6150 4050
-Connection ~ 6150 4050
-Wire Wire Line
-	6100 3400 6150 3400
-Wire Wire Line
-	6150 3400 6150 3600
-Connection ~ 6150 3600
 $Comp
 L power:GND #PWR0104
@@
 	1    0    0    -1
 $EndComp
+$Comp
+L 74xx:74LS32 U?
+U 4 1 5FA6D7A1
+P 5650 2950
+AR Path="/5F806563/5FA6D7A1" Ref="U?"  Part="4"
+AR Path="/5F806563/5F9E8365/5FA6D7A1" Ref="U14"  Part="4"
+F 0 "U14" H 5650 3275 50  0000 C CNN
+F 1 "74HCT32" H 5650 3184 50  0000 C CNN
+F 2 "Package_SO:SOIC-14_3.9x8.7mm_P1.27mm" H 5650 2950 50  0001 C CNN
+F 3 "http://www.ti.com/lit/gpn/sn74LS32" H 5650 2950 50  0001 C CNN
+	4    5650 2950
+	1    0    0    -1
+$EndComp
+Wire Wire Line
+	5350 3050 5250 3050
+Wire Wire Line
+	5250 3050 5250 2850
+Wire Wire Line
+	5350 2850 5250 2850
+Connection ~ 5250 2850
+Wire Wire Line
+	5250 2850 5150 2850
+Text GLabel 5150 2850 0    50   Input ~ 0
+SD_IRQ
+Text GLabel 6050 2950 2    50   Output ~ 0
+IRQ6
+Wire Wire Line
+	6050 2950 5950 2950
 Wire Bus Line
 	8700 1100 8700 1750

Commit message: Updated I/O board
Parts:
- removed U8: 74HC245, Package_SO:SOIC-20W_7.5x12.8mm_P1.27mm, symbol 74xx:74HC245
Connections:
- net GND: no longer U14.10, U14.9
- net ~D_EN: now reaches U14.8
- net ~WR_BUFFER renamed ~CS_BUFFER
- new net ~D_EN_3: U14.10, U14.9
- no-connect marks 5 -> 4
Other:
- moved on the sheet: U10, U11, U14A, U14B, U14C, U14D, U9
