File: KiCad/io_board/misc.sch (KiCad schematic (older format))
At the start: 10 parts, among them U6 27C512

Commit message: Worked on I/O board.
Parts:
- C16: footprint Capacitor_THT:CP_Radial_D6.3mm_P2.50mm -> Capacitor_THT:CP_Radial_D5.0mm_P2.00mm
Connections:
- net ~CS_DRVBUF: no longer names the net of U6.16 (D4)
- no-connect marks 3 -> 4
Changed lines of the file:
@@
 $Descr A4 11693 8268
 encoding utf-8
-Sheet 6 7
-Title ""
-Date ""
+Sheet 7 7
+Title "Mini8086 I/O board"
+Date "2020-11-05"
 Rev "1.0"
 Comp ""
@@
 F 0 "C16" H 9718 3546 50  0000 L CNN
 F 1 "47µ" H 9718 3455 50  0000 L CNN
-F 2 "Capacitor_THT:CP_Radial_D6.3mm_P2.50mm" H 9638 3350 50  0001 C CNN
+F 2 "Capacitor_THT:CP_Radial_D5.0mm_P2.00mm" H 9638 3350 50  0001 C CNN
 F 3 "~" H 9600 3500 50  0001 C CNN
 	1    9600 3500
@@
 ~RD
 Wire Wire Line
-	3700 2450 3800 2450
-Text GLabel 3800 2450 2    50   Output ~ 0
-~CS_DRVBUF
-Wire Wire Line
 	2800 3250 2800 3750
 Wire Wire Line
@@
 Connection ~ 6450 3750
 NoConn ~ 3700 2550
+NoConn ~ 3700 2450
 Wire Bus Line
 	2600 1850 2600 2650

Commit message: Working on IO board
Parts:
- C10, C11: footprint Capacitor_THT:C_Disc_D4.3mm_W1.9mm_P5.00mm -> Capacitor_SMD:C_1206_3216Metric
Changed lines of the file:
@@
 $Descr A4 11693 8268
 encoding utf-8
-Sheet 7 7
+Sheet 7 8
 Title "Mini8086 I/O board"
 Date "2020-11-05"
@@
 F 0 "C10" H 7015 3546 50  0000 L CNN
 F 1 "100n" H 7015 3455 50  0000 L CNN
-F 2 "Capacitor_THT:C_Disc_D4.3mm_W1.9mm_P5.00mm" H 6938 3350 50  0001 C CNN
+F 2 "Capacitor_SMD:C_1206_3216Metric" H 6938 3350 50  0001 C CNN
 F 3 "~" H 6900 3500 50  0001 C CNN
 	1    6900 3500
@@
 F 0 "C11" H 7465 3546 50  0000 L CNN
 F 1 "100n" H 7465 3455 50  0000 L CNN
-F 2 "Capacitor_THT:C_Disc_D4.3mm_W1.9mm_P5.00mm" H 7388 3350 50  0001 C CNN
+F 2 "Capacitor_SMD:C_1206_3216Metric" H 7388 3350 50  0001 C CNN
 F 3 "~" H 7350 3500 50  0001 C CNN
 	1    7350 3500

Commit message: Worked on I/O board.
Connections:
- net ~CS_I2C: now reaches U6.16 (D4)
- no-connect marks 4 -> 3
Other:
- note added: "I/O address decoder"
- note removed: "io address decoder"
- moved on the sheet: C10, C11, C12, C13, C14, C15, C16, C19, C20, U6

Commit message: Continued work on I/O board.
Parts:
- added C30, C31, C32, C33, C34, C35, C36, C38, C39: 100n, Capacitor_SMD:C_1206_3216Metric, symbol Device:C
- C12, C13, C14, C15, C19, C20: footprint Capacitor_THT:C_Disc_D4.3mm_W1.9mm_P5.00mm -> Capacitor_SMD:C_1206_3216Metric
Connections:
- net GND: now also C30.2, C31.2, C32.2, C33.2, C34.2, C35.2, C36.2, C38.2, C39.2
- net VCC: now also C30.1, C31.1, C32.1, C33.1, C34.1, C35.1, C36.1, C38.1, C39.1
Other:
- moved on the sheet: C10, C11, C12, C13, C14, C15, C16, C19, C20

Commit message: Worked on I/O board.
Connections:
- net ~CS_BUFFER renamed ~WR_BUFFER
Changed lines of the file:
@@
 	4650 2500 4050 2500
 Text GLabel 4650 2500 2    50   Output ~ 0
-~CS_BUFFER
+~WR_BUFFER
 Wire Wire Line
 	3250 3600 2800 3600

Commit message: Updated I/O board
Parts:
- removed C10: 100n, Capacitor_SMD:C_1206_3216Metric, symbol Device:C
- added C41: 100n, Capacitor_SMD:C_1206_3216Metric, symbol Device:C
Connections:
- net GND: now also C41.2
- net M_~IO: now also U6.26 (A13); no longer U6.1 (A15)
- net VCC: no longer C39.1
- net ~WR: now also U6.1 (A15); no longer U6.26 (A13)
- net ~WR_BUFFER renamed ~CS_BUFFER
- new net VCC3: C39.1, C41.1
Other:
- moved on the sheet: C19, C20, C30, C31, C32, C33, C34, C35, C36, C38, C39, U6
