File: KiCad/io_board/serial.sch (KiCad schematic (older format))
At the start: 2 parts

Commit message: Updated IO board schematics and board.
Parts:
- added C1, C2: 22p, Capacitor_THT:C_Disc_D3.0mm_W1.6mm_P2.50mm, symbol Device:C
- added C3, C4, C5, C6: 10µ, Capacitor_THT:CP_Radial_D5.0mm_P2.50mm, symbol Device:CP
- added J1: RS232, Connector_Dsub:DSUB-9_Male_Horizontal_P2.77x2.84mm_EdgePinOffset4.94mm_Housed_MountingHolesOffset7.48mm, symbol Connector:DB9_Male_MountingHoles
- added R1: 10M, Resistor_THT:R_Axial_DIN0207_L6.3mm_D2.5mm_P7.62mm_Horizontal, symbol Device:R_Small
- added R2: 470, Resistor_THT:R_Axial_DIN0207_L6.3mm_D2.5mm_P7.62mm_Horizontal, symbol Device:R_Small
- added R3: 3K3, Resistor_THT:R_Axial_DIN0207_L6.3mm_D2.5mm_P7.62mm_Horizontal, symbol Device:R
- added Y1: 8 MHz, Crystal:Crystal_HC49-U_Vertical, symbol Device:Crystal
- U1: renamed from U?; footprint Package_DIP:DIP-40_W15.24mm -> Package_DIP:DIP-40_W15.24mm_Socket_LongPads
- U2: renamed from U?; footprint (none) -> Package_DIP:DIP-16_W7.62mm_LongPads
Connections:
- net labels added: A0, A1, A2, A[0..19], CTS, D0, D1, D2, D3, D4, D5, D6, D7, D[0..7], GND, IRQ4, RESET, RTS, RX, TX, VCC, ~CS_UART, ~RD, ~WR
- wire segments 0 -> 88
- no-connect marks 0 -> 9
Other:
- moved on the sheet: U2

Commit message: Worked on I/O board.
Changed lines of the file:
@@
 encoding utf-8
 Sheet 2 7
-Title ""
-Date ""
+Title "Mini8086 I/O board"
+Date "2020-11-05"
 Rev "1.0"
 Comp ""
@@
 Wire Wire Line
 	3150 4800 2850 4800
-Text GLabel 2850 4800 0    50   Input ~ 0
+Text GLabel 2850 4800 0    50   Output ~ 0
 IRQ4
 $Comp

Commit message: Working on IO board
Parts:
- removed U1: 16550, Package_DIP:DIP-40_W15.24mm_Socket_LongPads, symbol Interface_UART:16550
- added U1: ST16C550CJ44, Package_LCC:PLCC-44_THT-Socket, symbol Mini8086:ST16C550CJ44
- added U16: MAX485E, Package_DIP:DIP-8_W7.62mm_LongPads, symbol Interface_UART:MAX485E
- C1, C2: value 22p -> 27p
- R1: value 10M -> 1M
- R2: value 470 -> 47
Other:
- moved on the sheet: C1, C2, C3, C4, C5, C6, J1, R1, R2, R3, U2, Y1

Commit message: Worked on I/O board.
Parts:
- R1, R2, R3: footprint Resistor_THT:R_Axial_DIN0207_L6.3mm_D2.5mm_P7.62mm_Horizontal -> Resistor_THT:R_Axial_DIN0207_L6.3mm_D2.5mm_P2.54mm_Vertical
Changed lines of the file:
@@
 F 0 "R2" V 2946 3100 50  0000 C CNN
 F 1 "47" V 2855 3100 50  0000 C CNN
-F 2 "Resistor_THT:R_Axial_DIN0207_L6.3mm_D2.5mm_P7.62mm_Horizontal" H 2750 3100 50  0001 C CNN
+F 2 "Resistor_THT:R_Axial_DIN0207_L6.3mm_D2.5mm_P2.54mm_Vertical" H 2750 3100 50  0001 C CNN
 F 3 "~" H 2750 3100 50  0001 C CNN
 	1    2750 3100
@@
 F 0 "R1" H 2091 2904 50  0000 R CNN
 F 1 "1M" H 2091 2995 50  0000 R CNN
-F 2 "Resistor_THT:R_Axial_DIN0207_L6.3mm_D2.5mm_P7.62mm_Horizontal" H 2150 2950 50  0001 C CNN
+F 2 "Resistor_THT:R_Axial_DIN0207_L6.3mm_D2.5mm_P2.54mm_Vertical" H 2150 2950 50  0001 C CNN
 F 3 "~" H 2150 2950 50  0001 C CNN
 	1    2150 2950
@@
 F 0 "R3" V 8843 2200 50  0000 C CNN
 F 1 "3K3" V 8934 2200 50  0000 C CNN
-F 2 "Resistor_THT:R_Axial_DIN0207_L6.3mm_D2.5mm_P7.62mm_Horizontal" V 8980 2200 50  0001 C CNN
+F 2 "Resistor_THT:R_Axial_DIN0207_L6.3mm_D2.5mm_P2.54mm_Vertical" V 8980 2200 50  0001 C CNN
 F 3 "~" H 9050 2200 50  0001 C CNN
 	1    9050 2200
@@
 D7
 $Comp
-L Mini8086:ST16C550CJ44 U1
-U 1 1 5FACF9F3
-P 4100 2600
-F 0 "U1" H 4100 2650 50  0000 C CNN
-F 1 "ST16C550CJ44" H 4100 2500 50  0000 C CNN
-F 2 "Package_LCC:PLCC-44_THT-Socket" H 4100 2600 50  0001 C CIN
-F 3 "" H 4100 2600 50  0001 C CNN
-	1    4100 2600
-	1    0    0    -1
-$EndComp
-$Comp
 L Interface_UART:MAX485E U16
 U 1 1 5FB33CEB
@@
 	1    0    0    -1
 $EndComp
+$Comp
+L Mini8086:ST16C550CJ44 U1
+U 1 1 5FC8676D
+P 4100 2600
+F 0 "U1" H 4100 2600 50  0000 C CNN
+F 1 "ST16C550CJ44" H 4100 2450 50  0000 C CNN
+F 2 "Package_LCC:PLCC-44_THT-Socket" H 4100 2600 50  0001 C CIN
+F 3 "" H 4100 2600 50  0001 C CNN
+	1    4100 2600
+	1    0    0    -1
+$EndComp

Commit message: Continued work on I/O board.
Parts:
- C1, C2: footprint Capacitor_THT:C_Disc_D3.0mm_W1.6mm_P2.50mm -> Capacitor_SMD:C_1206_3216Metric
- R1, R2, R3: footprint Resistor_THT:R_Axial_DIN0207_L6.3mm_D2.5mm_P2.54mm_Vertical -> Resistor_SMD:R_1206_3216Metric
- U2: footprint Package_DIP:DIP-16_W7.62mm_LongPads -> Package_SO:SOIC-16_3.9x9.9mm_P1.27mm
Connections:
- net XTAL2: now reaches R2.2, U1.19 (XTAL2)
- net XTAL1: now reaches C1.1, R1.2, U1.18 (XTAL1), Y1.2
Other:
- moved on the sheet: R2
Changed lines of the file:
@@
 F 0 "U2" H 6950 2550 50  0000 C CNN
 F 1 "MAX232" H 7300 1200 50  0000 C CNN
-F 2 "Package_DIP:DIP-16_W7.62mm_LongPads" H 7000 1250 50  0001 L CNN
+F 2 "Package_SO:SOIC-16_3.9x9.9mm_P1.27mm" H 7000 1250 50  0001 L CNN
 F 3 "http://www.ti.com/lit/ds/symlink/max232.pdf" H 6950 2400 50  0001 C CNN
 	1    6950 2300
@@
 L Device:R_Small R2
 U 1 1 5F8BA463
-P 2750 3100
-F 0 "R2" V 2946 3100 50  0000 C CNN
-F 1 "47" V 2855 3100 50  0000 C CNN
-F 2 "Resistor_THT:R_Axial_DIN0207_L6.3mm_D2.5mm_P2.54mm_Vertical" H 2750 3100 50  0001 C CNN
-F 3 "~" H 2750 3100 50  0001 C CNN
-	1    2750 3100
+P 2450 3100
+F 0 "R2" V 2646 3100 50  0000 C CNN
+F 1 "47" V 2555 3100 50  0000 C CNN
+F 2 "Resistor_SMD:R_1206_3216Metric" H 2450 3100 50  0001 C CNN
+F 3 "~" H 2450 3100 50  0001 C CNN
+	1    2450 3100
 	0    -1   -1   0
 $EndComp
@@
 F 0 "R1" H 2091 2904 50  0000 R CNN
 F 1 "1M" H 2091 2995 50  0000 R CNN
-F 2 "Resistor_THT:R_Axial_DIN0207_L6.3mm_D2.5mm_P2.54mm_Vertical" H 2150 2950 50  0001 C CNN
+F 2 "Resistor_SMD:R_1206_3216Metric" H 2150 2950 50  0001 C CNN
 F 3 "~" H 2150 2950 50  0001 C CNN
 	1    2150 2950
@@
 F 0 "C2" H 1765 3446 50  0000 L CNN
 F 1 "27p" H 1765 3355 50  0000 L CNN
-F 2 "Capacitor_THT:C_Disc_D3.0mm_W1.6mm_P2.50mm" H 1688 3250 50  0001 C CNN
+F 2 "Capacitor_SMD:C_1206_3216Metric" H 1688 3250 50  0001 C CNN
 F 3 "~" H 1650 3400 50  0001 C CNN
 	1    1650 3400
@@
 F 0 "C1" H 1315 3446 50  0000 L CNN
 F 1 "27p" H 1315 3355 50  0000 L CNN
-F 2 "Capacitor_THT:C_Disc_D3.0mm_W1.6mm_P2.50mm" H 1238 3250 50  0001 C CNN
+F 2 "Capacitor_SMD:C_1206_3216Metric" H 1238 3250 50  0001 C CNN
 F 3 "~" H 1200 3400 50  0001 C CNN
 	1    1200 3400
@@
 $EndComp
 Wire Wire Line
-	3100 3100 2850 3100
+	3100 3100 2550 3100
 Wire Wire Line
 	2150 2800 2150 2850
@@
 	2150 3100 2150 3050
 Wire Wire Line
-	2150 3100 2650 3100
+	2150 3100 2350 3100
 $Comp
 L Device:Crystal Y1
@@
 F 0 "R3" V 8843 2200 50  0000 C CNN
 F 1 "3K3" V 8934 2200 50  0000 C CNN
-F 2 "Resistor_THT:R_Axial_DIN0207_L6.3mm_D2.5mm_P2.54mm_Vertical" V 8980 2200 50  0001 C CNN
+F 2 "Resistor_SMD:R_1206_3216Metric" V 8980 2200 50  0001 C CNN
 F 3 "~" H 9050 2200 50  0001 C CNN
 	1    9050 2200
@@
 	1    0    0    -1
 $EndComp
+Text Label 2700 2800 0    50   ~ 0
+XTAL1
+Text Label 2700 3100 0    50   ~ 0
+XTAL2
 Wire Bus Line
 	2800 1950 2800 2200

Commit message: Updated I/O board
Parts:
- removed U16: MAX485E, Package_DIP:DIP-8_W7.62mm_LongPads, symbol Interface_UART:MAX485E
Changed lines of the file:
@@
 D7
-$Comp
-L Interface_UART:MAX485E U16
-U 1 1 5FB33CEB
-P 6950 5100
-F 0 "U16" H 6700 4500 50  0000 C CNN
-F 1 "MAX485E" H 7200 4500 50  0000 C CNN
-F 2 "Package_DIP:DIP-8_W7.62mm_LongPads" H 6950 4400 50  0001 C CNN
-F 3 "https://datasheets.maximintegrated.com/en/ds/MAX1487E-MAX491E.pdf" H 6950 5150 50  0001 C CNN
-	1    6950 5100
-	1    0    0    -1
-$EndComp
-$Comp
-L power:GND #PWR0106
-U 1 1 5FB411DC
-P 6950 5700
-F 0 "#PWR0106" H 6950 5450 50  0001 C CNN
-F 1 "GND" H 6955 5527 50  0000 C CNN
-F 2 "" H 6950 5700 50  0001 C CNN
-F 3 "" H 6950 5700 50  0001 C CNN
-	1    6950 5700
-	1    0    0    -1
-$EndComp
-$Comp
-L power:VCC #PWR0107
-U 1 1 5FB414A6
-P 6950 4600
-F 0 "#PWR0107" H 6950 4450 50  0001 C CNN
-F 1 "VCC" H 6965 4773 50  0000 C CNN
-F 2 "" H 6950 4600 50  0001 C CNN
-F 3 "" H 6950 4600 50  0001 C CNN
-	1    6950 4600
-	1    0    0    -1
-$EndComp
 $Comp
 L Mini8086:ST16C550CJ44 U1

Commit message: Worked on I/O board.
Parts:
- C3, C4, C5, C6: footprint Capacitor_THT:CP_Radial_D5.0mm_P2.50mm -> Capacitor_SMD:CP_Elec_4x3.9
Connections:
- no-connect marks 9 -> 13
Changed lines of the file:
@@
 F 0 "C3" H 6068 1596 50  0000 L CNN
 F 1 "10µ" H 6068 1505 50  0000 L CNN
-F 2 "Capacitor_THT:CP_Radial_D5.0mm_P2.50mm" H 5988 1400 50  0001 C CNN
+F 2 "Capacitor_SMD:CP_Elec_4x3.9" H 5988 1400 50  0001 C CNN
 F 3 "~" H 5950 1550 50  0001 C CNN
 	1    5950 1550
@@
 F 0 "C4" H 8018 1596 50  0000 L CNN
 F 1 "10µ" H 8018 1505 50  0000 L CNN
-F 2 "Capacitor_THT:CP_Radial_D5.0mm_P2.50mm" H 7938 1400 50  0001 C CNN
+F 2 "Capacitor_SMD:CP_Elec_4x3.9" H 7938 1400 50  0001 C CNN
 F 3 "~" H 7900 1550 50  0001 C CNN
 	1    7900 1550
@@
 F 0 "C6" H 8232 1504 50  0000 R CNN
 F 1 "10µ" H 8232 1595 50  0000 R CNN
-F 2 "Capacitor_THT:CP_Radial_D5.0mm_P2.50mm" H 8388 1400 50  0001 C CNN
+F 2 "Capacitor_SMD:CP_Elec_4x3.9" H 8388 1400 50  0001 C CNN
 F 3 "~" H 8350 1550 50  0001 C CNN
 	1    8350 1550
@@
 F 0 "C5" H 7982 3254 50  0000 R CNN
 F 1 "10µ" H 7982 3345 50  0000 R CNN
-F 2 "Capacitor_THT:CP_Radial_D5.0mm_P2.50mm" H 8138 3150 50  0001 C CNN
+F 2 "Capacitor_SMD:CP_Elec_4x3.9" H 8138 3150 50  0001 C CNN
 F 3 "~" H 8100 3300 50  0001 C CNN
 	1    8100 3300
@@
 Text Label 2700 3100 0    50   ~ 0
 XTAL2
+NoConn ~ 3950 4250
+NoConn ~ 3850 4250
+NoConn ~ 3750 4250
+NoConn ~ 3650 4250
 Wire Bus Line
 	2800 1950 2800 2200

Commit message: Updated I/O board
Connections:
- net RTS_5: now reaches U1.36 (~RTS~), U2.10 (T2IN)
- net TX_5: now reaches U1.13 (TX), U2.11 (T1IN)
- net RX_5: now reaches U1.11 (RX), U2.12 (R1OUT)
- net CTS_5: now reaches U1.40 (~CTS~), U2.9 (R2OUT)
- net RCLK: now reaches U1.10 (RCLK), U1.17 (~BAUDOUT~)
Changed lines of the file:
@@
 ~RD
 Wire Wire Line
-	5100 3800 5300 3800
-Wire Wire Line
-	5300 3800 5300 4000
-Wire Wire Line
-	5300 4000 5100 4000
+	5100 3800 5650 3800
+Wire Wire Line
+	5650 3800 5650 4000
+Wire Wire Line
+	5650 4000 5100 4000
 Wire Wire Line
 	5100 1400 5200 1400
@@
 NoConn ~ 3750 4250
 NoConn ~ 3650 4250
+Text Label 5150 1700 0    50   ~ 0
+CTS_5
+Text Label 5150 2200 0    50   ~ 0
+RTS_5
+Text Label 5150 2800 0    50   ~ 0
+RX_5
+Text Label 5150 2900 0    50   ~ 0
+TX_5
+Text Label 5250 4000 0    50   ~ 0
+RCLK
 Wire Bus Line
 	2800 1950 2800 2200
