File: KiCad/main/connector.sch (KiCad schematic (older format))
At the start: 14 parts, among them X2 Edge72-Mini8086

Commit message: Updated graphics adapter and main schematics + board.
Connections:
- net labels added: ~IO_DBG
- wire segments 106 -> 107
- no-connect marks 6 -> 5
Changed lines of the file:
@@
 A[0..19]
 NoConn ~ 4050 2200
-NoConn ~ 3100 2500
 NoConn ~ 3100 2400
 NoConn ~ 3100 2300
@@
 U 1 1 5F7F509D
 P 3550 3700
+AR Path="/5F7F509D" Ref="X2"  Part="1"
+AR Path="/5F7408B5/5F7F509D" Ref="X2"  Part="1"
 F 0 "X2" H 3575 5665 50  0000 C CNN
 F 1 "Edge72-Mini8086" H 3575 5574 50  0000 C CNN
@@
 Wire Wire Line
 	5700 4700 5700 4600
+Connection ~ 6100 4700
+Wire Wire Line
+	3100 2500 3000 2500
+Text GLabel 3000 2500 0    50   Input ~ 0
+~IO_DBG
 Wire Bus Line
 	2750 3300 2750 5300
 Wire Bus Line
 	4500 3700 4500 5300
-Connection ~ 6100 4700
 $EndSCHEMATC

Commit message: Updated KiCad VGA board and main board.
Parts:
- removed X2: Edge72-Mini8086, Mini8086:BUS_72, symbol main-rescue:Edge72-Mini8086
- added X2: Edge72, Mini8086:BUS_72, symbol Mini8086:Edge72
Connections:
- net labels added: IRQ1, NMI, TMR2
- net labels removed: IRQ2
- wire segments 107 -> 109
- no-connect marks 5 -> 3
Changed lines of the file:
@@
 	4400 3000 4050 3000
 Text GLabel 4400 3500 2    50   Input ~ 0
-IRQ2
+IRQ1
 Text GLabel 4400 3400 2    50   Input ~ 0
 IRQ3
@@
 A[0..19]
 NoConn ~ 4050 2200
-NoConn ~ 3100 2400
-NoConn ~ 3100 2300
 NoConn ~ 3100 2200
 NoConn ~ 3100 3100
@@
 Text GLabel 2550 2600 0    50   Input ~ 0
 PCLK
-$Comp
-L main-rescue:Edge72-Mini8086 X2
-U 1 1 5F7F509D
-P 3550 3700
-AR Path="/5F7F509D" Ref="X2"  Part="1"
-AR Path="/5F7408B5/5F7F509D" Ref="X2"  Part="1"
-F 0 "X2" H 3575 5665 50  0000 C CNN
-F 1 "Edge72-Mini8086" H 3575 5574 50  0000 C CNN
-F 2 "Mini8086:BUS_72" H 4100 3700 50  0001 C CNN
-F 3 "" H 4100 3700 50  0001 C CNN
-	1    3550 3700
-	1    0    0    -1
-$EndComp
 $Comp
 L Device:C C4
@@
 Text GLabel 3000 2500 0    50   Input ~ 0
 ~IO_DBG
+$Comp
+L Mini8086:Edge72 X2
+U 1 1 5F808933
+P 3550 3700
+F 0 "X2" H 3575 5665 50  0000 C CNN
+F 1 "Edge72" H 3575 5574 50  0000 C CNN
+F 2 "Mini8086:BUS_72" H 4100 3700 50  0001 C CNN
+F 3 "" H 4100 3700 50  0001 C CNN
+	1    3550 3700
+	1    0    0    -1
+$EndComp
+Wire Wire Line
+	3100 2400 2550 2400
+Wire Wire Line
+	3100 2300 3000 2300
 Wire Bus Line
 	2750 3300 2750 5300
 Wire Bus Line
 	4500 3700 4500 5300
+Text GLabel 2550 2400 0    50   Input ~ 0
+NMI
+Text GLabel 3000 2300 0    50   Input ~ 0
+TMR2
 $EndSCHEMATC

Commit message: Updated main system board schematics and board.
Parts:
- added C16, C17: 100n, Capacitor_THT:C_Disc_D4.3mm_W1.9mm_P5.00mm, symbol Device:C
- C11: value 10µ -> 100µ; footprint Capacitor_THT:CP_Radial_D4.0mm_P2.00mm -> Capacitor_THT:CP_Radial_D8.0mm_P3.50mm
- C12: value 10µ -> 47µ
Connections:
- net GND: now also C16.2, C17.2
- net VCC: now also C16.1, C17.1
Changed lines of the file:
@@
 $Descr A4 11693 8268
 encoding utf-8
-Sheet 5 5
-Title ""
+Sheet 5 6
+Title "Mini8086 main system board"
 Date ""
-Rev ""
+Rev "1.1"
 Comp ""
 Comment1 ""
@@
 P 10100 4450
 F 0 "C11" H 10218 4496 50  0000 L CNN
-F 1 "10µ" H 10218 4405 50  0000 L CNN
-F 2 "Capacitor_THT:CP_Radial_D4.0mm_P2.00mm" H 10138 4300 50  0001 C CNN
+F 1 "100µ" H 10218 4405 50  0000 L CNN
+F 2 "Capacitor_THT:CP_Radial_D8.0mm_P3.50mm" H 10138 4300 50  0001 C CNN
 F 3 "~" H 10100 4450 50  0001 C CNN
 	1    10100 4450
@@
 P 10500 4450
 F 0 "C12" H 10618 4496 50  0000 L CNN
-F 1 "10µ" H 10618 4405 50  0000 L CNN
+F 1 "47µ" H 10618 4405 50  0000 L CNN
 F 2 "Capacitor_THT:CP_Radial_D4.0mm_P2.00mm" H 10538 4300 50  0001 C CNN
 F 3 "~" H 10500 4450 50  0001 C CNN
@@
 Wire Wire Line
 	3100 2300 3000 2300
-Wire Bus Line
-	2750 3300 2750 5300
-Wire Bus Line
-	4500 3700 4500 5300
 Text GLabel 2550 2400 0    50   Input ~ 0
 NMI
 Text GLabel 3000 2300 0    50   Input ~ 0
 TMR2
+$Comp
+L Device:C C17
+U 1 1 5F8A088B
+P 10500 5700
+F 0 "C17" H 10615 5746 50  0000 L CNN
+F 1 "100n" H 10615 5655 50  0000 L CNN
+F 2 "Capacitor_THT:C_Disc_D4.3mm_W1.9mm_P5.00mm" H 10538 5550 50  0001 C CNN
+F 3 "~" H 10500 5700 50  0001 C CNN
+	1    10500 5700
+	1    0    0    -1
+$EndComp
+$Comp
+L Device:C C16
+U 1 1 5F8A0891
+P 10100 5700
+F 0 "C16" H 10215 5746 50  0000 L CNN
+F 1 "100n" H 10215 5655 50  0000 L CNN
+F 2 "Capacitor_THT:C_Disc_D4.3mm_W1.9mm_P5.00mm" H 10138 5550 50  0001 C CNN
+F 3 "~" H 10100 5700 50  0001 C CNN
+	1    10100 5700
+	1    0    0    -1
+$EndComp
+Wire Wire Line
+	10500 5450 10500 5550
+Wire Wire Line
+	10500 5450 10100 5450
+Wire Wire Line
+	10100 5450 10100 5550
+Wire Wire Line
+	10500 5950 10500 5850
+Wire Wire Line
+	10500 5950 10100 5950
+Wire Wire Line
+	10100 5950 10100 5850
+$Comp
+L power:GND #PWR063
+U 1 1 5F8C489C
+P 10500 6050
+F 0 "#PWR063" H 10500 5800 50  0001 C CNN
+F 1 "GND" H 10505 5877 50  0000 C CNN
+F 2 "" H 10500 6050 50  0001 C CNN
+F 3 "" H 10500 6050 50  0001 C CNN
+	1    10500 6050
+	1    0    0    -1
+$EndComp
+$Comp
+L power:VCC #PWR062
+U 1 1 5F8D4561
+P 10500 5350
+F 0 "#PWR062" H 10500 5200 50  0001 C CNN
+F 1 "VCC" H 10515 5523 50  0000 C CNN
+F 2 "" H 10500 5350 50  0001 C CNN
+F 3 "" H 10500 5350 50  0001 C CNN
+	1    10500 5350
+	1    0    0    -1
+$EndComp
+Wire Wire Line
+	10500 6050 10500 5950
+Connection ~ 10500 5950
+Wire Wire Line
+	10500 5350 10500 5450
+Connection ~ 10500 5450
+Wire Bus Line
+	4500 3700 4500 5300
+Wire Bus Line
+	2750 3300 2750 5300
 $EndSCHEMATC
