File: KiCad/main/main.kicad_pcb (KiCad board)
At the start: 4 copper layers, 160 x 100.1 mm, 51 parts, among them SW1 SW_Push, U1 74HC245, U10 8254, U11 8259, U12 27C512, U13 74HC32, U14 74HC245, U15 74HC08, U2 8284, U3 74HC245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

Commit message: Minor changes on CPU boards
Routing:
- net GND: vias 48 -> 47
