File: KiCad/main/main.sch (KiCad schematic (older format))
At the start: 0 parts

Commit message: Updated main system board schematics and board.
Changed lines of the file:
@@
 $Descr A4 11693 8268
 encoding utf-8
-Sheet 1 5
-Title ""
+Sheet 1 6
+Title "Mini8086 main system board"
 Date ""
-Rev ""
+Rev "1.1"
 Comp ""
 Comment1 ""
@@
 F1 "connector.sch" 50
 $EndSheet
+$Sheet
+S 7000 1000 1000 1000
+U 5F8BB07A
+F0 "glue logic" 50
+F1 "glue logic.sch" 50
+$EndSheet
 $EndSCHEMATC

Commit message: Minor changes on CPU boards
Changed lines of the file:
@@
 S 7000 1000 1000 1000
 U 5F8BB07A
-F0 "glue logic" 50
-F1 "glue logic.sch" 50
+F0 "misc" 50
+F1 "misc.sch" 50
 $EndSheet
 $EndSCHEMATC
