File: KiCad/info_board/info_board.sch (KiCad schematic (older format))
At the start: 1 part, among them X1 Edge72

Commit message: Updated KiCad versioning information in schematics. Fixed button wrong pinout in backplane. Added missing files to git.
Parts:
- X1: symbol Mini8086:Edge72 -> info_board-rescue:Edge72-Mini8086
Changed lines of the file:
@@
 $EndComp
 $Comp
-L Mini8086:Edge72 X1
+L info_board-rescue:Edge72-Mini8086 X1
 U 1 1 5F982738
 P 4100 3850
