File: KiCad/led_board/led_board.sch (KiCad schematic (older format))
At the start: 8 parts, among them X1 Edge72

Commit message: Updated KiCad versioning information in schematics. Fixed button wrong pinout in backplane. Added missing files to git.
Parts:
- X1: symbol Mini8086:Edge72 -> led_board-rescue:Edge72-Mini8086
Changed lines of the file:
@@
 encoding utf-8
 Sheet 1 4
-Title ""
+Title "Mini8086 LED board"
 Date ""
-Rev ""
+Rev "1.1"
 Comp ""
 Comment1 ""
@@
 $EndDescr
 $Comp
-L Mini8086:Edge72 X1
+L led_board-rescue:Edge72-Mini8086 X1
 U 1 1 5FD2F4CE
 P 3500 4000
