File: KiCad/main_v2/cpu.sch (KiCad schematic (older format))
At the start: 6 parts, among them U1 SN74ALVC164245, U2 SN74ALVC164245, U4 8086

Commit message: Fixed PCB bugs in main V2
Connections:
- net GND: now also U2.1 (1DIR), U2.24 (2DIR)
- net VCC36: no longer U2.1 (1DIR), U2.24 (2DIR)
Changed lines of the file:
@@
 	1    0    0    -1
 $EndComp
-Text GLabel 7750 4000 0    50   Input ~ 0
-VCC36
-Text GLabel 7750 5900 0    50   Input ~ 0
-VCC36
 Text GLabel 7350 4550 0    50   Input ~ 0
 ~BHE~_S7
@@
 Wire Wire Line
 	7650 5650 7650 5550
-Wire Wire Line
-	7650 5750 7300 5750
-Wire Wire Line
-	7300 5750 7300 6200
 Connection ~ 7650 5750
 $Comp
 L power:GND #PWR0101
 U 1 1 5FF4B1C8
-P 7300 6200
-F 0 "#PWR0101" H 7300 5950 50  0001 C CNN
-F 1 "GND" H 7305 6027 50  0000 C CNN
-F 2 "" H 7300 6200 50  0001 C CNN
-F 3 "" H 7300 6200 50  0001 C CNN
-	1    7300 6200
+P 7650 6250
+F 0 "#PWR0101" H 7650 6000 50  0001 C CNN
+F 1 "GND" H 7655 6077 50  0000 C CNN
+F 2 "" H 7650 6250 50  0001 C CNN
+F 3 "" H 7650 6250 50  0001 C CNN
+	1    7650 6250
 	1    0    0    -1
 $EndComp
 Text Notes 6700 3250 0    50   ~ 0
 0 = output (B -> A)\n1 = input (A -> B)\n
+Wire Wire Line
+	7750 5900 7650 5900
+Wire Wire Line
+	7650 5900 7650 5750
+$Comp
+L power:GND #PWR0110
+U 1 1 6014334C
+P 7750 4000
+F 0 "#PWR0110" H 7750 3750 50  0001 C CNN
+F 1 "GND" V 7750 3800 50  0000 C CNN
+F 2 "" H 7750 4000 50  0001 C CNN
+F 3 "" H 7750 4000 50  0001 C CNN
+	1    7750 4000
+	0    1    1    0
+$EndComp
+Wire Wire Line
+	7650 6250 7650 5900
 Wire Bus Line
 	9750 4000 9750 4350
@@
 Wire Bus Line
 	3600 1900 3600 3950
+Connection ~ 7650 5900
 $EndSCHEMATC
