File: KiCad/main_v2/main.kicad_pcb (KiCad board)
At the start: 4 copper layers, 98.8 x 100.1 mm, 69 parts, among them J1 JTAG, SW1 Reset, U1 SN74ALVC164245, U10 8254, U11 8259, U12 SN74ALVC164245, U2 SN74ALVC164245, U3 LM317, U4 8086, U5 EPM570T144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

Commit message: Fixed PCB bugs in main V2
Parts:
- U3: footprint Package_TO_SOT_SMD:SOT-223-3_TabPin2 -> Package_TO_SOT_SMD:TO-252-2
- moved R4 1.14 mm to (125.0, 122.7)
- moved U3 0.25 mm to (132.1, 123.4)
Connections:
- U2 pad 1: VCC36 -> GND
- U2 pad 24: VCC36 -> GND
Routing:
- net VCC36: track 369.4 -> 362.5 mm, vias 32 -> 27
- net Net-(R4-Pad2): track 16.7 -> 15.5 mm
- net TDO: track 85.0 -> 86.2 mm
- net /CPLD/~CPLD_RESET: track 61.7 -> 62.8 mm
- net GND: vias 169 -> 170
Other:
- board text added: "Rev. 2.1 2020-2021"
- board text removed: "Rev. 2.0 2020-2021"

Commit message: Minor changes on CPU boards
Routing:
- net GND: vias 170 -> 160
