File: KiCad/main_v2/connector.sch (KiCad schematic (older format))
At the start: 37 parts, among them U3 LM317, X2 Edge72

Commit message: Fixed PCB bugs in main V2
Parts:
- U3: footprint Package_TO_SOT_SMD:SOT-223-3_TabPin2 -> Package_TO_SOT_SMD:TO-252-2
Changed lines of the file:
@@
 F 0 "U3" H 5550 2092 50  0000 C CNN
 F 1 "LM317" H 5550 2001 50  0000 C CNN
-F 2 "Package_TO_SOT_SMD:SOT-223-3_TabPin2" H 5550 2100 50  0001 C CIN
+F 2 "Package_TO_SOT_SMD:TO-252-2" H 5550 2100 50  0001 C CIN
 F 3 "http://www.ti.com/lit/ds/symlink/lm317.pdf" H 5550 1850 50  0001 C CNN
 	1    5550 1850

Commit message: Added documentation.
Other:
- note added: "Bottom"
- note added: "Left"
- note added: "Right"
- note added: "Top"
Changed lines of the file:
@@
 Wire Bus Line
 	1800 2450 1800 4450
+Text Notes 3750 2900 0    100  ~ 0
+Bottom
+Text Notes 1300 2900 0    100  ~ 0
+Top
+Text Notes 2500 4950 0    100  ~ 0
+Right
+Text Notes 2550 750  0    100  ~ 0
+Left
 $EndSCHEMATC
