File: KiCad/io_board_v2/connector.sch (KiCad schematic (older format))
At the start: 2 parts, among them U4 74HCT04, X1 Edge72

Commit message: Fixed wrong Mini-DIN 6 footprint.
Other:
- moved on the sheet: U4G
Changed lines of the file:
@@
 Title "Mini8086 I/O board"
 Date "2020-11-05"
-Rev "2.0"
+Rev "1.2"
 Comp ""
 Comment1 ""
@@
 L 74xx:74HC04 U4
 U 7 1 5F904FC3
-P 8550 4050
-F 0 "U4" H 8780 4096 50  0000 L CNN
-F 1 "74HCT04" H 8780 4005 50  0000 L CNN
-F 2 "Package_SO:SOIC-14_3.9x8.7mm_P1.27mm" H 8550 4050 50  0001 C CNN
-F 3 "https://assets.nexperia.com/documents/data-sheet/74HC_HCT04.pdf" H 8550 4050 50  0001 C CNN
-	7    8550 4050
+P 6900 3950
+F 0 "U4" H 7130 3996 50  0000 L CNN
+F 1 "74HCT04" H 7130 3905 50  0000 L CNN
+F 2 "Package_SO:SOIC-14_3.9x8.7mm_P1.27mm" H 6900 3950 50  0001 C CNN
+F 3 "https://assets.nexperia.com/documents/data-sheet/74HC_HCT04.pdf" H 6900 3950 50  0001 C CNN
+	7    6900 3950
 	1    0    0    -1
 $EndComp
@@
 L power:GND #PWR059
 U 1 1 5F90625F
-P 8550 4550
-F 0 "#PWR059" H 8550 4300 50  0001 C CNN
-F 1 "GND" H 8555 4377 50  0000 C CNN
-F 2 "" H 8550 4550 50  0001 C CNN
-F 3 "" H 8550 4550 50  0001 C CNN
-	1    8550 4550
+P 6900 4450
+F 0 "#PWR059" H 6900 4200 50  0001 C CNN
+F 1 "GND" H 6905 4277 50  0000 C CNN
+F 2 "" H 6900 4450 50  0001 C CNN
+F 3 "" H 6900 4450 50  0001 C CNN
+	1    6900 4450
 	1    0    0    -1
 $EndComp
@@
 L power:VCC #PWR058
 U 1 1 5F90653C
-P 8550 3550
-F 0 "#PWR058" H 8550 3400 50  0001 C CNN
-F 1 "VCC" H 8565 3723 50  0000 C CNN
-F 2 "" H 8550 3550 50  0001 C CNN
-F 3 "" H 8550 3550 50  0001 C CNN
-	1    8550 3550
-	1    0    0    -1
-$EndComp
+P 6900 3450
+F 0 "#PWR058" H 6900 3300 50  0001 C CNN
+F 1 "VCC" H 6915 3623 50  0000 C CNN
+F 2 "" H 6900 3450 50  0001 C CNN
+F 3 "" H 6900 3450 50  0001 C CNN
+	1    6900 3450
+	1    0    0    -1
+$EndComp
