File: KiCad/io_board_v2/SD drive.sch (KiCad schematic (older format))
At the start: 36 parts, among them J3 SD_Card, J4 JTAG, U12 AMS1117-3.3, U13 SN74LVC245A, U15 SN74LVC8T245PWR, U6 MicroSD_SPI_CD, U7 EPM240T100, X2 20 MHz

Commit message: Fixed I/O board issues.
Parts:
- R12, R13, R15: value 100 -> 120
Changed lines of the file:
@@
 ~RD
 Entry Wire Line
-	1300 2500 1200 2400
-Text GLabel 1100 2350 0    50   Input ~ 0
+	1700 2500 1600 2400
+Text GLabel 1500 2350 0    50   Input ~ 0
 A[0..19]
-Text Label 1400 2500 0    50   ~ 0
+Text Label 1800 2500 0    50   ~ 0
 A0
 Wire Wire Line
@@
 Connection ~ 5500 1600
 Entry Wire Line
-	1300 2600 1200 2500
-Text Label 1400 2600 0    50   ~ 0
+	1700 2600 1600 2500
+Text Label 1800 2600 0    50   ~ 0
 A1
 Wire Wire Line
@@
 	3750 3550 3650 3550
 Wire Bus Line
-	1100 2350 1200 2350
+	1500 2350 1600 2350
 Text Label 3950 3700 0    50   ~ 0
 AL3
@@
 	2300 2300 1900 2300
 Wire Wire Line
-	1300 2500 2300 2500
-Wire Wire Line
-	1300 2600 2300 2600
+	1700 2500 2300 2500
+Wire Wire Line
+	1700 2600 2300 2600
 Text GLabel 2300 2900 0    50   Input ~ 0
 VCC3
@@
 P 7050 6000
 F 0 "R12" V 7246 6000 50  0000 C CNN
-F 1 "100" V 7155 6000 50  0000 C CNN
+F 1 "120" V 7155 6000 50  0000 C CNN
 F 2 "Resistor_SMD:R_1206_3216Metric" H 7050 6000 50  0001 C CNN
 F 3 "~" H 7050 6000 50  0001 C CNN
@@
 P 7050 6200
 F 0 "R13" V 6850 6200 50  0000 C CNN
-F 1 "100" V 6950 6200 50  0000 C CNN
+F 1 "120" V 6950 6200 50  0000 C CNN
 F 2 "Resistor_SMD:R_1206_3216Metric" H 7050 6200 50  0001 C CNN
 F 3 "~" H 7050 6200 50  0001 C CNN
@@
 P 7050 5000
 F 0 "R15" V 7246 5000 50  0000 C CNN
-F 1 "100" V 7155 5000 50  0000 C CNN
+F 1 "120" V 7155 5000 50  0000 C CNN
 F 2 "Resistor_SMD:R_1206_3216Metric" H 7050 5000 50  0001 C CNN
 F 3 "~" H 7050 5000 50  0001 C CNN
@@
 	9050 5200 8800 5200
 Wire Bus Line
-	1200 2350 1200 2500
+	1600 2350 1600 2500
 Wire Bus Line
 	1200 4850 1200 5600
