File: KiCad/io_board_v2/SD misc.sch (KiCad schematic (older format))
At the start: 2 parts, among them U8 74HCT04, U9 SN74LVC245A

Commit message: Fixed I/O board issues.
Other:
- moved on the sheet: U8A, U8B, U8C, U8D, U8E, U8F, U8G, U9
